Commit message: restructured the whole package

File: src/robot_description/urdf/robot.urdf (robot description, URDF)
Before this commit: robot ur10e_robot, 45 links, 44 joints
Links:
- link base_link_inertia: geometry collision mesh filename=package://robot_description/meshes/ur10e/collision/base.stl; visual mesh filename=package://robot_description/meshes/ur10e/visual/base.dae
- link camera_link: geometry collision box size=0.02505 0.09 0.025; visual mesh filename=package://robot_description/meshes/camera_stl/d435.dae
- link clamp_base_link: geometry collision mesh filename=package://robot_description/meshes/camera_stl/clamp_base.stl scale=0.001 0.001 0.001; visual mesh filename=package://robot_description/meshes/camera_stl/clamp_base.stl scale=0.001 0.001 0.001
- link clamp_stem_link: geometry collision mesh filename=package://robot_description/meshes/camera_stl/clamp_stem.stl scale=0.001 0.001 0.001; visual mesh filename=package://robot_description/meshes/camera_stl/clamp_stem.stl scale=0.001 0.001 0.001
- link forearm_link: geometry collision mesh filename=package://robot_description/meshes/ur10e/collision/forearm.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; visual mesh filename=package://robot_description/meshes/ur10e/visual/forearm.dae
- link fts_link: geometry collision mesh filename=package://robot_description/meshes/on_robot_ft/onrobot_hexe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; visual mesh filename=package://robot_description/meshes/on_robot_ft/onrobot_hexe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
- link rg2_gripper_base_link: geometry collision mesh filename=package://robot_description/meshes/on_robot_rg2/collision/b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; visual mesh filename=package://robot_description/meshes/on_robot_rg2/visual/base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
- link rg2_gripper_left_inner_finger: geometry collision mesh filename=package://robot_description/meshes/on_robot_rg2/collision/i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; visual mesh filename=package://robot_description/meshes/on_robot_rg2/visual/inne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
- link rg2_gripper_left_inner_knuckle: geometry collision mesh filename=package://robot_description/meshes/on_robot_rg2/collision/i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; visual mesh filename=package://robot_description/meshes/on_robot_rg2/visual/inne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
- link rg2_gripper_left_outer_knuckle: geometry collision mesh filename=package://robot_description/meshes/on_robot_rg2/collision/o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; visual mesh filename=package://robot_description/meshes/on_robot_rg2/visual/oute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
- link rg2_gripper_right_inner_finger: geometry collision mesh filename=package://robot_description/meshes/on_robot_rg2/collision/i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; visual mesh filename=package://robot_description/meshes/on_robot_rg2/visual/inne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
- link rg2_gripper_right_inner_knuckle: geometry collision mesh filename=package://robot_description/meshes/on_robot_rg2/collision/i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; visual mesh filename=package://robot_description/meshes/on_robot_rg2/visual/inne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
- link rg2_gripper_right_outer_knuckle: geometry collision mesh filename=package://robot_description/meshes/on_robot_rg2/collision/o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; visual mesh filename=package://robot_description/meshes/on_robot_rg2/visual/oute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
- link shoulder_link: geometry collision mesh filename=package://robot_description/meshes/ur10e/collision/shoulder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; visual mesh filename=package://robot_description/meshes/ur10e/visual/shoulder.dae
- link upper_arm_link: geometry collision mesh filename=package://robot_description/meshes/ur10e/collision/upperarm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; visual mesh filename=package://robot_description/meshes/ur10e/visual/upperarm.dae
- link ur10e_nozzle_for_tape: geometry collision mesh filename=package://robot_description/meshes/Nozzle_for_tape.stl scale=0.001 0.001 0.001; visual mesh filename=package://robot_description/meshes/Nozzle_for_tape.stl scale=0.001 0.001 0.001
- link wrist_1_link: geometry collision mesh filename=package://robot_description/meshes/ur10e/collision/wrist1.s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; visual mesh filename=package://robot_description/meshes/ur10e/visual/wrist1.dae
- link wrist_2_link: geometry collision mesh filename=package://robot_description/meshes/ur10e/collision/wrist2.s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; visual mesh filename=package://robot_description/meshes/ur10e/visual/wrist2.dae
- link wrist_3_link: geometry collision mesh filename=package://robot_description/meshes/ur10e/collision/wrist3.s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; visual mesh filename=package://robot_description/meshes/ur10e/visual/wrist3.dae
