Commit message: rviz  connection with issac sim done

File: src/moveit_config/config/ur.ros2_control.xacro (robot description, xacro)
@@ -5,6 +5,5 @@
         <ros2_control name="${name}" type="system">
             <hardware>
-                <!-- By default, set up controllers for simulation. This won't work on real hardware -->
-                <plugin>mock_components/GenericSystem</plugin>
+                <plugin>topic_based_ros2_control/TopicBasedSystem</plugin>
             </hardware>
             <joint name="shoulder_pan_joint">

File: src/robot_description/urdf/complete_ws.urdf (robot description, URDF)
Before this commit: robot ur, 59 links, 58 joints
Joints:
- joint base_joint: origin xyz=1.63 0.83 0.928 rpy=0 0 3.14 -> xyz=1.63 0.83 0.928 rpy=0 0 1.57
